File: Termometer_test.kicad_pcb (KiCad board)
At the start: 2 copper layers, 55 x 115 mm, 7 parts

Commit message: Add files via upload
Parts:
- added H1: MountingHole, MountingHole:MountingHole_3.2mm_M3_DIN965_Pad, F.Cu at (139.0, 53.0)
- added H2: MountingHole, MountingHole:MountingHole_3.2mm_M3_DIN965_Pad, F.Cu at (86.0, 156.0)
- added H3: MountingHole, MountingHole:MountingHole_3.2mm_M3_DIN965_Pad, F.Cu at (139.0, 156.0)
- added H4: MountingHole, MountingHole:MountingHole_3.2mm_M3_DIN965_Pad, F.Cu at (86.0, 53.0)
- moved TrimPot1 26.4 mm to (108.0, 90.0)
- moved Batteri1 17.0 mm to (134.0, 94.8)
- moved Temp1 17.0 mm to (134.0, 140.0)
- moved Temp2 17.0 mm to (134.0, 121.0)
Routing:
- net Net-(LCD1-V0): track 63.3 -> 35.0 mm
- net Net-(A1-VSYS): track 225.8 -> 203.6 mm
- net Net-(A1-GPIO7): track 91.2 -> 79.7 mm
- net Net-(A1-GPIO14): track 75.5 -> 81.4 mm, vias 2 -> 1
- net Net-(A1-GPIO19): track 86.9 -> 90.4 mm
Other:
- board size 55 x 115 mm -> 65 x 115 mm
