File: Termometer_test.kicad_sch (KiCad schematic)
At the start: 7 parts, among them U1 DS18B20, U2 DS18B20

Commit message: Add files via upload
Parts:
- removed RV1: 10k, symbol Device:R_Potentiometer
- removed U1, U2: DS18B20, Package_TO_SOT_THT:TO-92_Inline, symbol Sensor_Temperature:DS18B20
- removed V1: 4.5, symbol Simulation_SPICE:VDC
- added Batteri1: Screw_Terminal_01x02, TerminalBlock:TerminalBlock_MaiXu_MX126-5.0-02P_1x02_P5.00mm, symbol Connector:Screw_Terminal_01x02
- added Temp1, Temp2: Screw_Terminal_01x03, TerminalBlock:TerminalBlock_MaiXu_MX126-5.0-03P_1x03_P5.00mm, symbol Connector:Screw_Terminal_01x03
- added TrimPot1: R_Potentiometer_Trim, Potentiometer_THT:Potentiometer_Runtron_RM-065_Vertical, symbol Device:R_Potentiometer_Trim
- LCD1: footprint (none) -> Termometer_test:LCD
- R1: value 4.7k -> R; footprint (none) -> Resistor_THT:R_Axial_DIN0204_L3.6mm_D1.6mm_P7.62mm_Horizontal
Connections:
- net GND: now also A1.13 (GND), A1.18 (GND), A1.23 (GND), A1.28 (GND), A1.3 (GND), A1.38 (GND), A1.8 (GND), Batteri1.2 (Pin_2), Temp1.2 (Pin_2), Temp2.2 (Pin_2), TrimPot1.3
- net at A1.39 (VSYS), LCD1.2 (Vdd), R1.1: now also Batteri1.1 (Pin_1), Temp1.1 (Pin_1), Temp2.1 (Pin_1), TrimPot1.1
- net at LCD1.3 (V0): now also TrimPot1.2
- net at R1.2: now also A1.10 (GPIO7), Temp1.3 (Pin_3), Temp2.3 (Pin_3); no longer A1.21 (GPIO16)
- net at LCD1.11 (DB4): now also A1.16 (GPIO12); no longer A1.12 (GPIO9)
- net at LCD1.12 (DB5): now also A1.12 (GPIO9); no longer A1.16 (GPIO12)
- net at LCD1.13 (DB6): now also A1.15 (GPIO11); no longer A1.14 (GPIO10)
- net at LCD1.14 (DB7): now also A1.14 (GPIO10); no longer A1.15 (GPIO11)
- net at LCD1.6 (E): now also A1.25 (GPIO19); no longer A1.17 (GPIO13)
Other:
- note removed: "Databus"
- note removed: "Pullup resistor"

Commit message: Add files via upload
Parts:
- added H1, H2, H3, H4: MountingHole, MountingHole:MountingHole_3.2mm_M3_DIN965_Pad, symbol Mechanical:MountingHole
